File: hardware/connectors.kicad_sch (KiCad schematic)
At the start: 37 parts, among them J1 Conn_01x02, J2 uFL ant, J3 SMA ant, J4 uFL ant, J5 SMA ant, J6 Conn_01x02, J7 USB_A, J8 FTSH-107-01-L-D-K, J9 XIAO ESP32S3 Sense, U4 FT231XS-U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

Commit message: Finished routing
Parts:
- added H1, H2, H3, H4: MountingHole_Pad, MountingHole:MountingHole_3mm_Pad_Via, symbol Mechanical:MountingHole_Pad
Connections:
- net CAN+: now also D6.1 (A1); no longer D6.2 (A2)
- net CAN-: now also D6.2 (A2); no longer D6.1 (A1)
- net D+: now also D3.1 (A1)
- net D-: now also D3.2 (A2)
- net GND_EXT: now also H4.1
- net PROG_SWCLK: now also D11.4 (K); no longer D11.3 (K)
- net PROG_SWDIO: now also D11.3 (K); no longer D11.4 (K)
- net d+: no longer D3.1 (A1)
- net d-: no longer D3.2 (A2)
- no-connect marks 22 -> 25
Other:
- note added: "Mounting Holes"

Commit message: Some smaller fixes and final aesthetic changes
Parts:
- added TP10: VN_RX, TestPoint:TestPoint_Pad_D1.0mm, symbol Connector:TestPoint
- added TP11: D-, TestPoint07:TestPoint_Pad_D0.7mm, symbol Connector:TestPoint
- added TP12: D+, TestPoint07:TestPoint_Pad_D0.7mm, symbol Connector:TestPoint
- added TP9: VN_TX, TestPoint:TestPoint_Pad_D1.0mm, symbol Connector:TestPoint
- H1, H2, H3: footprint MountingHole:MountingHole_3mm_Pad_Via -> MountingHole:MountingHole_3mm
Connections:
- net D+: now also TP12.1
- net D-: now also TP11.1
- net VN_RX: now also TP9.1
- net VN_TX: now also TP10.1
Other:
- company: Author: -> Author: Kacper Pawlak
- moved on the sheet: C16, C24, C25, D3, D4, D5, R13, R14, R21, U6

Commit message: little changes with traces and 3D models visibility
Changed lines of the file:
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@@
 	)
 	(hierarchical_label "VN_TX"
-		(shape output)
+		(shape input)
 		(at 162.56 88.9 0)
 		(effects

Commit message: Updated BOM
Parts:
- C12, C14, C16: Mouser No (none) -> 81-GCM188R71H103KA7J
- C24, C25: Mouser -- -> dnp; Mouser No (none) -> ---
- D10, D9: Manufacturer_Part_Number STS232050B751 -> (none)
- D11: Manufacturer_Part_Number ESDS304DBVR -> (none)
- D15, D16, D2, D8: Mouser No (none) -> 576-SMF5.0A
- D3: Mouser No (none) -> 511-ESDAVLC6-2BLY
- D4, D5: Mouser No (none) -> 710-150060BS55040
- D6: value 27V/420W -> 28V/350W; Mouser https://www.mouser.pl/ProductDetail/Micro-Commercial-Compon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 -> https://www.mouser.pl/ProductDetail/Nexperia/PESD5V0L2BT-QR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; Mouser No (none) -> 771-PESD5V0L2BT-QR
- D7: Mouser No (none) -> 863-NSVRB751V40T1G
- FB1: Mouser No (none) -> 875-MI0805K400R-10
- H1, H2, H3, H4: Mouser No (none) -> ---
- J1, J6: value Conn_01x02 -> strainrelief; Manufacturer_Part_Number strain relief -> (none)
- J2, J4: Mouser No (none) -> 712-CONUFL001-SMD-T
- J3, J5: Mouser No (none) -> 471-SMACONNECTOR
- J7: Mouser No (none) -> 490-UJ2-AV-4-TH
- J8: Manufacturer_Part_Number FTSH-107-01-L-D-K -> (none)
- J9: Mouser No (none) -> ---; Mouser Part Number . -> (none)
- R10, R11: Mouser No (none) -> 667-ERJ-3RED27R0V
- R12: Mouser No (none) -> 603-AC0603FR-0710KL
- R13, R14: Mouser No (none) -> 71-RCS0603330RJNEA
- R21: Mouser No (none) -> 71-CRCW06031K00FKEE71-CRCW06031K00FKEE
- TP10, TP11, TP12, TP9: Mouser (none) -> ---; Mouser No (none) -> ---
- U4: Height 1.753 -> (none); Manufacturer_Name FTDI Chip -> (none); Manufacturer_Part_Number FT231XS-U -> (none); Mouser https://www.mouser.pl/ProductDetail/FTDI/FT231XS-R?qs=Gp1Yz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 -> https://www.mouser.pl/ProductDetail/FTDI/FT231XS-U?qs=Gp1Yz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; Mouser No (none) -> 895-FT231XS-U; Mouser Part Number 895-FT231XS-U -> (none); Mouser Price/Stock https://www.mouser.co.uk/ProductDetail/FTDI/FT231XS-U?qs=Gp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 -> (none)
- U5: Mouser No (none) -> 621-API7721FSB-13
- U6: value AQY284S -> AQY284SX; Mouser No (none) -> 769-AQY284SX
