File: hardware/mcu.kicad_sch (KiCad schematic)
At the start: 10 parts, among them U2 STM32G0C1KCTxN

Commit message: Updated BOM
Parts:
- R6, R7, R8: Mouser No (none) -> 603-RC0603FR-7W33RL
- TP4, TP5, TP6, TP7: Mouser (none) -> ---; Mouser No (none) -> ---
- U2: Mouser No (none) -> 511-STM32G0C1KCT6N
