File: hardware/power.kicad_sch (KiCad schematic)
At the start: 17 parts, among them Q2 SI2347DS-T1-GE3, U7 NCP565D2T33R4G, U8 SI06W8-05

Commit message: Finished routing
Parts:
- removed C21: 47uF+, 47uCapPolarized:EEE1AA220WR, symbol Device:C_Polarized_Small
- removed U8: SI06W8-05, DCisoconv:SI06W805, symbol SI06W8-05:SI06W8-05
- added C21: 20uF, 20uF5Vcap:GRM31x, symbol Device:C_Small
- added TP1: 24V_TestPoint, TestPoint:TestPoint_Pad_D1.0mm, symbol Connector:TestPoint
- added TP2: 5V_TestPoint, TestPoint:TestPoint_Pad_D1.0mm, symbol Connector:TestPoint
- added TP3: 3V3_TestPoint, TestPoint:TestPoint_Pad_D1.0mm, symbol Connector:TestPoint
- added U8: RSH3-2405S_H2, DCisoconv:RSH32405SH2, symbol RSH3-2405S_H2:RSH3-2405S_H2
- C17: value 2.2uF -> 10uF; footprint Capacitor_SMD:C_1206_3216Metric_Pad1.33x1.80mm_HandSolder -> 10uF24Vcap:CAPC6050X550N; Mouser https://www.mouser.pl/ProductDetail/Murata-Electronics/GRM3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 -> https://www.mouser.pl/ProductDetail/KEMET/C2220C226M5R2CAUT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
- L1: value 10uH -> 3.9uH; footprint inductor:VLS3010 -> inductor:RLS397; Mouser https://www.mouser.pl/ProductDetail/TDK/VLS3010CX-100M-1?qs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 -> https://eu.mouser.com/ProductDetail/RECOM-Power/RLS-397?qs=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
Connections:
- net +3.3V: now also TP3.1
- net +5V: now also C21.1, TP2.1, U8.8 (+VOUT)
- net GND: now also C21.2, U8.9 (-VOUT)
- net GND_EXT: now also U8.1 (-VIN)
- net at C18.1, C19.1, L1.2: now also TP1.1, U8.14 (+VIN)
- no-connect marks 0 -> 1
Other:
- moved on the sheet: F1

Commit message: Some smaller fixes and final aesthetic changes
Parts:
- removed C17: 10uF, 10uF24Vcap:CAPC6050X550N, symbol Device:C_Small
- removed C18: 2.2uF, Capacitor_SMD:C_1206_3216Metric_Pad1.33x1.80mm_HandSolder, symbol Device:C_Small
- added C27, C28, C29, C30, C31, C32: 10uF, Capacitor_SMD:C_1206_3216Metric, symbol Device:C_Small
Connections:
- net GND_EXT: now also C27.2, C28.2, C29.2, C30.2, C31.2, C32.2
- net at D13.1 (K), L1.1, Q2.2 (S): now also C27.1, C28.1, C29.1
- net at C19.1, L1.2, TP1.1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: now also C30.1, C31.1, C32.1
Other:
- company: Author: -> Author: Kacper Pawlak
- moved on the sheet: C19, C20, C21, C22, C23, D12, D13, D14, F1, L1, Q2, R15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

Commit message: Updated BOM
Parts:
- C19, C20: Mouser No (none) -> 767-LS1808N151K302NT
- C21: Mouser No (none) -> 81-GRM31CR61A476ME5L
- C22, C23: Mouser https://www.mouser.pl/ProductDetail/Murata-Electronics/GRM188R60J476ME15D?qs=sGAEpiMZZMvsSlwiRhF8qmz4GBGiC1clmSm1Iyhv5VVtC0STJ%2F5n0A%3D%3D -> https://www.mouser.pl/ProductDetail/Murata-Electronics/GRM188R60J476ME15J?qs=5aG0NVq1C4w8O78wi%2F2m1g%3D%3D; Mouser No (none) -> 81-GRM188R60J476ME5J
- C27, C28, C29, C30, C31, C32: Mouser No (none) -> 81-GRM31CD71H106KE1L
- D12: Mouser No (none) -> 576-SMF26CA
- D13: Mouser No (none) -> 863-SZMMSZ4697T1G
- D14: Mouser No (none) -> 710-150060BS55040
- F1: Mouser No (none) -> 576-0467.250NR
- L1: Mouser No (none) -> 919-RLS-397
- Q2: Mouser No (none) -> 78-SI2347DS-T1-BE3; Mouser Part Number 78-SI2347DS-T1-GE3 -> (none); Mouser Price/Stock https://www.mouser.pl/ProductDetail/Vishay-Semiconductors/S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 -> (none)
- R15: Mouser No (none) -> 660-RK73B1JTTD104J
- R16: Mouser No (none) -> 71-RCS0603330RJNEA
- TP1, TP2, TP3: Mouser (none) -> ---; Mouser No (none) -> ---
- U7: value NCP565D2T33R4G -> 863-NCP565D2T33R4G; Mouser No (none) -> 863-NCP565D2T33R4G
- U8: Mouser No (none) -> 919-RSH3-2405S/H2; Mouser Part Number 919-RSH3-2405S/H2 -> (none)
